File: kicad/usb-instrument/isolation.kicad_sch (KiCad schematic)
At the start: 6 parts, among them U4 ISO6742, U8 TEA 1-0505

Commit message: begin layout
Parts:
- U8: footprint TEA 1_TRP -> Converter_DCDC:Converter_DCDC_TRACO_TEA1-xxxx_THT
Connections:
- net VCC: now also R19.2; no longer R19.1
- net at U4.7 (EN1): now also R19.1; no longer R19.2
Other:
- moved on the sheet: C10, C9, R18, R19
