File: kicad/usb-instrument/output_stage.kicad_sch (KiCad schematic)
At the start: 28 parts, among them Q5 BS170, Q6 BSS84, Q7 BS170, Q8 BS170, U12 LM321, U13 LM321

Commit message: begin layout
Parts:
- D5, D6, D7: footprint (none) -> LED_SMD:LED_1206_3216Metric
- TP17: footprint (none) -> TestPoint:TestPoint_Pad_D2.5mm
Changed lines of the file:
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@@
 			)
 		)
-		(property "Footprint" ""
+		(property "Footprint" "TestPoint:TestPoint_Pad_D2.5mm"
 			(at 96.52 114.3 0)
 			(hide yes)
@@
 			)
 		)
-		(property "Footprint" ""
+		(property "Footprint" "LED_SMD:LED_1206_3216Metric"
 			(at 184.15 82.55 0)
 			(hide yes)
@@
 			)
 		)
-		(property "Footprint" ""
+		(property "Footprint" "LED_SMD:LED_1206_3216Metric"
 			(at 261.62 82.55 0)
 			(hide yes)
@@
 			)
 		)
-		(property "Footprint" ""
+		(property "Footprint" "LED_SMD:LED_1206_3216Metric"
 			(at 223.52 82.55 0)
 			(hide yes)
