File: kicad/usb-instrument/usb-instrument.kicad_pcb (KiCad board)
At the start: 2 copper layers, 100 x 100 mm, 57 parts, among them Q5 BS170, Q6 BSS84, Q7 BS170, Q8 BS170, U1 XIAO-ESP32-C3-DIP, U11 ISO6742, U12 LM321, U13 LM321, U2 ADS131M02IRUKR, U3 LM317_SOT-223, U4 ISO6742, U6 ISO6742, U7 ISO6742, U8 TEA 1-0505, U9 TLV172IDCK

Commit message: begin layout
Parts:
- removed R16, R17: 100k, Resistor_SMD:R_0805_2012Metric_Pad1.20x1.40mm_HandSolder
- removed R20, R21, R22, R23, R24, R25: 4.7k, Resistor_SMD:R_0805_2012Metric_Pad1.20x1.40mm_HandSolder
- removed U11, U6, U7: ISO6742, Package_SO:SOIC-16W_7.5x10.3mm_P1.27mm
- added C1: 10n, Capacitor_SMD:C_0805_2012Metric_Pad1.18x1.45mm_HandSolder, F.Cu at (123.1, 126.3)
- added C2: 10n, Capacitor_SMD:C_0805_2012Metric_Pad1.18x1.45mm_HandSolder, F.Cu at (129.5, 126.5)
- added C20: 220n, Capacitor_SMD:C_0805_2012Metric_Pad1.18x1.45mm_HandSolder, F.Cu at (73.1, 65.8)
- added C21: 10u, Capacitor_SMD:C_0805_2012Metric_Pad1.18x1.45mm_HandSolder, F.Cu at (78.2, 63.9)
- added C22: 1u, Capacitor_SMD:C_0805_2012Metric_Pad1.18x1.45mm_HandSolder, F.Cu at (57.2, 105.8)
- added C3: 47p (optional), Capacitor_SMD:C_0805_2012Metric_Pad1.18x1.45mm_HandSolder, F.Cu at (133.4, 96.1)
- added D5: LED, LED_SMD:LED_1206_3216Metric, F.Cu at (80.9, 132.0)
- added D6: LED, LED_SMD:LED_1206_3216Metric, F.Cu at (80.7, 144.2)
- added D7: LED, LED_SMD:LED_1206_3216Metric, F.Cu at (80.7, 147.6)
- added FB1: FerriteBead, Inductor_SMD:L_0603_1608Metric_Pad1.05x0.95mm_HandSolder, F.Cu at (58.2, 103.1)
- added J1: USB_B_Micro, Connector_USB:USB_Micro-B_Amphenol_10103594-0001LF_Horizontal, F.Cu at (52.2, 70.4)
- added J2: USB_C_Receptacle_USB2.0_14P, Connector_USB:USB_C_Receptacle_G-Switch_GT-USB-7010ASV, F.Cu at (52.9, 59.3)
- added R1: 1k, Resistor_SMD:R_0805_2012Metric_Pad1.20x1.40mm_HandSolder, F.Cu at (122.2, 129.2)
- added R2: 1k, Resistor_SMD:R_0805_2012Metric_Pad1.20x1.40mm_HandSolder, F.Cu at (124.1, 129.2)
- added R3: 1k, Resistor_SMD:R_0805_2012Metric_Pad1.20x1.40mm_HandSolder, F.Cu at (130.4, 129.4)
- added R4: 1k, Resistor_SMD:R_0805_2012Metric_Pad1.20x1.40mm_HandSolder, F.Cu at (128.4, 129.4)
- added R5: 5k1, Resistor_SMD:R_0805_2012Metric_Pad1.20x1.40mm_HandSolder, F.Cu at (61.9, 57.7)
- added R6: 5k1, Resistor_SMD:R_0805_2012Metric_Pad1.20x1.40mm_HandSolder, F.Cu at (61.9, 60.6)
- added R7: 22, Resistor_SMD:R_0805_2012Metric_Pad1.20x1.40mm_HandSolder, F.Cu at (134.9, 106.4)
- added R8: 10k, Resistor_SMD:R_0805_2012Metric_Pad1.20x1.40mm_HandSolder, F.Cu at (67.9, 73.9)
- added R9: 10k, Resistor_SMD:R_0805_2012Metric_Pad1.20x1.40mm_HandSolder, F.Cu at (127.7, 119.8)
- added TP1: MCP_RX, TestPoint:TestPoint_Pad_D2.5mm, F.Cu at (70.9, 73.3)
- added TP17: TestPoint, TestPoint:TestPoint_Pad_D2.5mm, F.Cu at (64.3, 112.3)
- added TP2: MCP_TX, TestPoint:TestPoint_Pad_D2.5mm, F.Cu at (71.0, 69.1)
- added U5: MCP2221AxSL, Package_SO:SOIC-14_3.9x8.7mm_P1.27mm, F.Cu at (63.2, 71.2)
- added Y1: XO32, Crystal:Crystal_SMD_7050-4Pin_7.0x5.0mm, F.Cu at (127.4, 115.4)
- C11, C14, C16: value 100n -> 10u
- C12: value 100n -> 220n
- C15: value 100n -> 100u; footprint Capacitor_SMD:C_0805_2012Metric_Pad1.18x1.45mm_HandSolder -> Capacitor_SMD:CP_Elec_6.3x5.7
- U2: footprint Xiao:WQFN20_ADS131_TEX -> Footprints:WQFN20_ADS131_TEX
- U8: footprint Xiao:TEA 1_TRP -> Converter_DCDC:Converter_DCDC_TRACO_TEA1-xxxx_THT
- moved C13 67.7 mm to (127.6, 111.5), turned to 180 degrees
- moved U3 60.0 mm to (108.1, 113.6)
- moved C4 56.3 mm to (101.7, 115.9), turned to 180 degrees
- moved R14 52.2 mm to (102.7, 112.5), turned to 90 degrees
- moved R15 50.7 mm to (100.7, 112.4), turned to -90 degrees
- moved U1 48.5 mm to (108.7, 60.3), turned to 90 degrees
- moved C5 47.6 mm to (113.5, 113.6), turned to 90 degrees
- moved C17 44.7 mm to (55.9, 113.0)
- moved R34 43.2 mm to (65.3, 138.6)
- moved R36 43.2 mm to (65.3, 144.5)
- moved R37 43.2 mm to (65.3, 147.5)
- moved R35 43.2 mm to (65.3, 141.6)
- moved C15 43.0 mm to (86.0, 59.5), turned to 90 degrees
- moved C16 41.7 mm to (132.8, 106.4), turned to -90 degrees
- moved C18 41.1 mm to (59.5, 117.0)
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Connections:
- net Net-(U13--) renamed /OUTPUT_STAGE/VDAC
- C12 pad 1: VCCQ -> Net-(U5-VUSB)
- C12 pad 2: GNDA -> GND
- C13 pad 1: VCC -> /ESP_3.3V
- C13 pad 2: GND -> GNDA
- C14 pad 1: VCCQ -> /OUTPUT_STAGE/5V_LEDS
- C15 pad 1: VCC -> VCCQ
- C15 pad 2: GND -> GNDA
- C16 pad 1: VCCQ -> /INPUT_STAGE/5V_OP
- C5 pad 1: /INPUT_STAGE/3.3V -> /INPUT_STAGE/AVDD
- C6 pad 1: /INPUT_STAGE/3.3V -> /INPUT_STAGE/AVDD
- C8 pad 1: /INPUT_STAGE/3.3V -> /ESP_3.3V
- Q6 pad 2: Net-(D5-A) -> /OUTPUT_STAGE/5V_LEDS
- Q6 pad 3: VCCQ -> Net-(D5-A)
- R14 pad 1: /INPUT_STAGE/3.3V -> /INPUT_STAGE/AVDD
- R19 pad 1: VCC -> Net-(U4-EN1)
- R19 pad 2: Net-(U4-EN1) -> VCC
- R26 pad 1: /ISOLATION/OUTG -> /GPIO5
- R30 pad 1: /ISOLATION/OUTD -> /GPIO2
- R34 pad 1: /ISOLATION/OUTE -> /GPIO3
- R36 pad 1: /ISOLATION/OUTF -> /GPIO4
- U1 pad 1: unconnected-(U1-GPIO2_A0_D0-Pad1) -> /GPIO2
- U1 pad 10: /ISOLATION/OUTA_2 -> /ESP_MISO
- U1 pad 11: /ISOLATION/INA -> /ESP_MOSI
- U1 pad 12: unconnected-(U1-3V3-Pad12) -> /ESP_3.3V
- U1 pad 13: GND -> GNDA
- U1 pad 14: VCC -> VCCQ
- U1 pad 2: unconnected-(U1-GPIO3_A1_D1-Pad2) -> /GPIO3
- U1 pad 3: unconnected-(U1-GPIO4_A2_D2-Pad3) -> /GPIO4
- U1 pad 4: /ISOLATION/ING -> /GPIO5
- U1 pad 5: /ISOLATION/INF -> /GPIO6
- U1 pad 6: /ISOLATION/INE -> /GPIO7
- U1 pad 7: /ISOLATION/IND -> /ESP_TX
- U1 pad 8: /ISOLATION/INC -> /ESP_RX
- U1 pad 9: /ISOLATION/INB -> /ESP_SCK
- U13 pad 5: VCCQ -> /OUTPUT_STAGE/5V_LEDS
- U2 pad 1: /INPUT_STAGE/V_PD -> /INPUT_STAGE/AIN0P
- U2 pad 11: unconnected-(U2-DRDY-Pad11) -> /GPIO6
- U2 pad 12: /INPUT_STAGE/SCLK -> /ESP_SCK
- U2 pad 13: /INPUT_STAGE/DOUT -> /ESP_MISO
- U2 pad 14: /INPUT_STAGE/DIN -> /ESP_MOSI
- U2 pad 18: /INPUT_STAGE/3.3V -> /ESP_3.3V
- U2 pad 19: /INPUT_STAGE/3.3V -> /INPUT_STAGE/AVDD
- U2 pad 2: GNDA -> /INPUT_STAGE/AIN0N
- U2 pad 3: /INPUT_STAGE/R_SENSE -> /INPUT_STAGE/AIN1N
- U2 pad 4: GNDA -> /INPUT_STAGE/AIN1P
- U2 pad 9: Net-(U2-SYNC/RESET) -> /GPIO7
- U3 pad 2: /INPUT_STAGE/3.3V -> /INPUT_STAGE/AVDD
- U4 pad 12: /INPUT_STAGE/DOUT -> /ESP_TX
- U4 pad 13: /INPUT_STAGE/SCLK -> /ISOLATION/OUTB
- U4 pad 14: /INPUT_STAGE/DIN -> /ESP_RX
- U4 pad 3: /ISOLATION/INA -> /MCP_TX
- U4 pad 5: /ISOLATION/OUTA_2 -> /MCP_RX
- U9 pad 5: VCCQ -> /INPUT_STAGE/5V_OP

Commit message: geroutet
Parts:
- added R10: 10k, Resistor_SMD:R_0805_2012Metric_Pad1.20x1.40mm_HandSolder, F.Cu at (138.5, 104.1)
- moved R36 100.3 mm to (120.9, 61.1), turned to 180 degrees
- moved R34 99.5 mm to (120.9, 56.1), turned to 180 degrees
- moved R30 92.7 mm to (120.9, 58.6), turned to 180 degrees
- moved R26 55.5 mm to (103.8, 89.2), turned to 180 degrees
- moved R27 53.3 mm to (103.6, 91.1), turned to 180 degrees
- moved C17 51.8 mm to (103.7, 93.1), turned to 180 degrees
- moved C18 49.3 mm to (100.1, 89.1), turned to 180 degrees
- moved R31 48.9 mm to (100.0, 101.2)
- moved U12 45.9 mm to (100.0, 92.2), turned to -90 degrees
- moved R28 43.3 mm to (97.2, 90.2), turned to -90 degrees
- moved R13 37.4 mm to (108.1, 121.4), turned to -90 degrees
- moved C22 37.3 mm to (94.2, 101.3), turned to 90 degrees
- moved TP17 35.8 mm to (93.5, 91.5), turned to 180 degrees
- moved FB1 35.0 mm to (93.2, 104.0), turned to 0 degrees
- moved D4 34.5 mm to (100.0, 120.0), turned to 180 degrees
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Connections:
- R1 pad 1: /INPUT_STAGE/V_PD -> /INPUT_STAGE/R_SENSE
- R26 pad 1: /GPIO5 -> /GPIO10
- R3 pad 1: /INPUT_STAGE/R_SENSE -> /INPUT_STAGE/V_PD
- R30 pad 1: /GPIO2 -> /GPIO4
- R36 pad 1: /GPIO4 -> /GPIO5
- R9 pad 1: GNDA -> /ESP_3.3V
- U1 pad 1: /GPIO2 -> /ESP_MOSI
- U1 pad 10: /ESP_MISO -> /SYNC/RESET
- U1 pad 11: /ESP_MOSI -> /GPIO10
- U1 pad 6: /GPIO7 -> /ESP_MISO
- U2 pad 9: /GPIO7 -> /SYNC/RESET
Routing:
- net Net-(Q7-G): track 0.00 -> 92.5 mm, vias 0 -> 2
- net Net-(Q8-G): track 0.00 -> 82.5 mm, vias 0 -> 2
- net /ESP_3.3V: track 0.00 -> 80.5 mm, vias 0 -> 4
- net /GPIO10: track 0.00 -> 59.8 mm, vias 0 -> 1
- net /ESP_MOSI: track 0.00 -> 58.2 mm
- net Net-(Q5-S): track 0.00 -> 57.1 mm
- net GNDA: track 0.00 -> 56.8 mm, vias 0 -> 220
- net Net-(Q5-G): track 0.00 -> 55.3 mm, vias 0 -> 2
- net /GPIO6: track 0.00 -> 51.7 mm, vias 0 -> 1
- net /ESP_RX: track 0.00 -> 51.0 mm, vias 0 -> 1
- net /SYNC/RESET: track 0.00 -> 46.4 mm
- net VCCQ: track 0.00 -> 46.1 mm, vias 0 -> 11
- net /ESP_MISO: track 0.00 -> 42.9 mm
- net /INPUT_STAGE/V_PD: track 0.00 -> 42.1 mm
- net /INPUT_STAGE/R_SENSE: track 0.00 -> 40.4 mm
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- added copper zone on B.Cu, net GND
- added copper zone on F.Cu, net GND
- added copper zone on In1.Cu, net GND
- added copper zone on B.Cu, net GNDA
- added copper zone on F.Cu, net GNDA
- added copper zone on In1.Cu, net GNDA
- added copper zone on In2.Cu, net VCC
- added copper zone on In2.Cu, net VCCQ
Other:
- copper layers 2 -> 4

Commit message: vias + logo
Parts:
- added G***: LOGO, LOGO, F.Cu at (61.9, 116.0)
Routing:
- net Net-(Q8-G): track 82.5 -> 97.1 mm
- net GNDA: vias 220 -> 259
- net GND: vias 5 -> 20

Commit message: smal fixes
Routing:
- net /ESP_3.3V: track 80.5 -> 99.0 mm, vias 4 -> 5
- net GNDA: track 56.8 -> 61.3 mm, vias 259 -> 264
- net /INPUT_STAGE/AIN1N: track 3.25 -> 5.19 mm
- net /INPUT_STAGE/AIN1P: track 4.87 -> 6.78 mm
