File: kicad/usb-instrument/usb-instrument.kicad_sch (KiCad schematic)
At the start: 14 parts, among them J1 USB_B_Micro, J2 USB_C_Receptacle_USB2.0_14P, U1 XIAO-ESP32-C3-DIP, U5 MCP2221AxSL

Commit message: begin layout
Parts:
- C12: footprint (none) -> Capacitor_SMD:C_0805_2012Metric_Pad1.18x1.45mm_HandSolder
- J2: footprint (none) -> Connector_USB:USB_C_Receptacle_G-Switch_GT-USB-7010ASV
- R5, R6, R8: footprint (none) -> Resistor_SMD:R_0805_2012Metric_Pad1.20x1.40mm_HandSolder
- TP1, TP2: footprint (none) -> TestPoint:TestPoint_Pad_D2.5mm
Changed lines of the file:
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@@
 			)
 		)
-		(property "Footprint" ""
+		(property "Footprint" "Resistor_SMD:R_0805_2012Metric_Pad1.20x1.40mm_HandSolder"
 			(at 52.07 47.498 90)
 			(hide yes)
@@
 			)
 		)
-		(property "Footprint" ""
+		(property "Footprint" "Connector_USB:USB_C_Receptacle_G-Switch_GT-USB-7010ASV"
 			(at 36.83 53.34 0)
 			(hide yes)
@@
 			)
 		)
-		(property "Footprint" ""
+		(property "Footprint" "Resistor_SMD:R_0805_2012Metric_Pad1.20x1.40mm_HandSolder"
 			(at 52.07 44.958 90)
 			(hide yes)
@@
 			)
 		)
-		(property "Footprint" ""
+		(property "Footprint" "TestPoint:TestPoint_Pad_D2.5mm"
 			(at 73.66 144.78 0)
 			(hide yes)
@@
 			)
 		)
-		(property "Footprint" ""
+		(property "Footprint" "Resistor_SMD:R_0805_2012Metric_Pad1.20x1.40mm_HandSolder"
 			(at 41.91 133.858 90)
 			(hide yes)
@@
 			)
 		)
-		(property "Footprint" ""
+		(property "Footprint" "TestPoint:TestPoint_Pad_D2.5mm"
 			(at 73.66 147.32 0)
 			(hide yes)
@@
 			)
 		)
-		(property "Footprint" ""
+		(property "Footprint" "Capacitor_SMD:C_0805_2012Metric_Pad1.18x1.45mm_HandSolder"
 			(at 57.4548 119.38 0)
 			(hide yes)

Commit message: geroutet
Connections:
- net GPIO2 is gone; now on net ESP_MOSI: U1.1 (GPIO2_A0_D0)
- net GPIO7 is gone; now on net ESP_MISO: U1.6 (GPIO7_D5_SCL)
- net ESP_MISO: no longer U1.10 (GPIO9_D9_MISO)
- net ESP_MOSI: no longer U1.11 (GPIO10_D10_MOSI)
- new net GPIO10: U1.11 (GPIO10_D10_MOSI)
- new net SYNC/RESET: U1.10 (GPIO9_D9_MISO)
Other:
- note added: "Strapping pins: GPIO2 - MOSI (should be high impedance input) GPIO8 - SCLK (should be high impedance input) GPIO9 - SYNC/RESET (pulled high)"
- note removed: "TODO Strapping pins"
Changed lines of the file:
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@@
 	(generator_version "10.0")
 	(paper "A4")
-	(text "TODO Strapping pins"
+	(text "Strapping pins: GPIO2 - MOSI (should be high impedance input)\n		 		GPIO8 - SCLK (should be high impedance input)\n		 		GPIO9 - SYNC/RESET			(pulled high)\n				"
 		(exclude_from_sim no)
-		(at 172.466 137.922 0)
+		(at 217.932 139.7 0)
 		(effects
 			(font
 				(size 1.27 1.27)
 			)
+			(justify right)
 		)
 	)
@@
 	(wire
 		(pts
-			(xy 161.29 99.06) (xy 168.91 99.06)
+			(xy 158.75 99.06) (xy 168.91 99.06)
 		)
 		(stroke
@@
 	(wire
 		(pts
-			(xy 215.9 76.2) (xy 207.01 76.2)
+			(xy 218.44 76.2) (xy 207.01 76.2)
 		)
 		(stroke
@@
 	(wire
 		(pts
-			(xy 161.29 91.44) (xy 168.91 91.44)
+			(xy 158.75 91.44) (xy 168.91 91.44)
 		)
 		(stroke
@@
 	(wire
 		(pts
-			(xy 161.29 80.01) (xy 168.91 80.01)
+			(xy 158.75 80.01) (xy 168.91 80.01)
 		)
 		(stroke
@@
 	(wire
 		(pts
-			(xy 207.01 91.44) (xy 217.17 91.44)
+			(xy 207.01 91.44) (xy 219.71 91.44)
 		)
 		(stroke
@@
 	(wire
 		(pts
-			(xy 208.28 80.01) (xy 207.01 80.01)
+			(xy 210.82 80.01) (xy 207.01 80.01)
 		)
 		(stroke
@@
 	(wire
 		(pts
-			(xy 161.29 95.25) (xy 168.91 95.25)
+			(xy 158.75 95.25) (xy 168.91 95.25)
 		)
 		(stroke
@@
 	(wire
 		(pts
-			(xy 161.29 87.63) (xy 168.91 87.63)
+			(xy 158.75 87.63) (xy 168.91 87.63)
 		)
 		(stroke
@@
 	(wire
 		(pts
-			(xy 217.17 87.63) (xy 207.01 87.63)
+			(xy 219.71 87.63) (xy 207.01 87.63)
 		)
 		(stroke
@@
 	(wire
 		(pts
-			(xy 217.17 83.82) (xy 207.01 83.82)
+			(xy 219.71 83.82) (xy 207.01 83.82)
 		)
 		(stroke
@@
 	(wire
 		(pts
-			(xy 207.01 99.06) (xy 217.17 99.06)
+			(xy 207.01 99.06) (xy 219.71 99.06)
 		)
 		(stroke
@@
 	(wire
 		(pts
-			(xy 161.29 83.82) (xy 168.91 83.82)
+			(xy 158.75 83.82) (xy 168.91 83.82)
 		)
 		(stroke
@@
 	(wire
 		(pts
-			(xy 217.17 95.25) (xy 207.01 95.25)
+			(xy 219.71 95.25) (xy 207.01 95.25)
 		)
 		(stroke
@@
 	(wire
 		(pts
-			(xy 161.29 76.2) (xy 168.91 76.2)
+			(xy 158.75 76.2) (xy 168.91 76.2)
 		)
 		(stroke
@@
 		)
 	)
-	(label "ESP_MISO"
-		(at 226.06 106.68 0)
-		(effects
-			(font
-				(size 1.27 1.27)
-			)
-			(justify left bottom)
-		)
-	)
 	(label "5V_ISO"
 		(at 227.33 34.29 0)
@@
 	)
 	(label "ESP_SCK"
-		(at 217.17 95.25 180)
+		(at 219.71 95.25 180)
 		(effects
 			(font
@@
 		)
 	)
-	(label "GPIO7"
-		(at 226.06 128.27 0)
-		(effects
-			(font
-				(size 1.27 1.27)
-			)
-			(justify left bottom)
-		)
-	)
 	(label "D+"
 		(at 96.52 64.77 180)
@@
 		)
 	)
-	(label "ESP_MISO"
-		(at 217.17 91.44 180)
-		(effects
-			(font
-				(size 1.27 1.27)
-			)
-			(justify right bottom)
-		)
-	)
 	(label "ESP_RX"
 		(at 143.51 96.52 180)
@@
 	)
 	(label "GPIO5"
-		(at 161.29 87.63 0)
+		(at 227.33 66.04 0)
 		(effects
 			(font
@@
 		)
 	)
-	(label "GPIO6"
-		(at 161.29 91.44 0)
+	(label "GPIO5"
+		(at 158.75 87.63 0)
 		(effects
 			(font
@@
 		)
 	)
-	(label "ESP_RX"
-		(at 217.17 99.06 180)
+	(label "GPIO6"
+		(at 158.75 91.44 0)
 		(effects
 			(font
 				(size 1.27 1.27)
 			)
-			(justify right bottom)
+			(justify left bottom)
 		)
 	)
-	(label "VBUS"
-		(at 90.17 24.13 0)
+	(label "ESP_RX"
+		(at 219.71 99.06 180)
 		(effects
 			(font
 				(size 1.27 1.27)
 			)
-			(justify left bottom)
+			(justify right bottom)
 		)
 	)
-	(label "GPIO2"
-		(at 227.33 60.96 0)
+	(label "VBUS"
+		(at 90.17 24.13 0)
 		(effects
 			(font
@@
 	)
 	(label "ESP_3.3V"
-		(at 217.17 83.82 180)
+		(at 219.71 83.82 180)
 		(effects
 			(font
@@
 		)
 	)
-	(label "ESP_MOSI"
-		(at 217.17 87.63 180)
+	(label "GPIO10"
+		(at 219.71 87.63 180)
 		(effects
 			(font
@@
 		)
 	)
-	(label "GPIO5"
-		(at 227.33 69.85 0)
+	(label "SYNC{slash}RESET"
+		(at 219.71 91.44 180)
 		(effects
 			(font
 				(size 1.27 1.27)
 			)
-			(justify left bottom)
+			(justify right bottom)
 		)
 	)
-	(label "GPIO4"
-		(at 227.33 66.04 0)
+	(label "MCP_TX"
+		(at 105.41 96.52 0)
 		(effects
 			(font
@@
 		)
 	)
-	(label "GPIO7"
-		(at 161.29 95.25 0)
+	(label "5V_ISO"
+		(at 146.05 24.13 180)
 		(effects
 			(font
 				(size 1.27 1.27)
 			)
-			(justify left bottom)
+			(justify right bottom)
 		)
 	)
-	(label "MCP_TX"
-		(at 105.41 96.52 0)
+	(label "MCP_RX"
+		(at 105.41 107.95 0)
 		(effects
 			(font
@@
 		)
 	)
-	(label "5V_ISO"
-		(at 146.05 24.13 180)
+	(label "MCP_TX"
+		(at 73.66 142.24 180)
 		(effects
 			(font
@@
 		)
 	)
-	(label "MCP_RX"
-		(at 105.41 107.95 0)
+	(label "GPIO3"
+		(at 158.75 80.01 0)
 		(effects
 			(font
@@
 		)
 	)
-	(label "MCP_TX"
-		(at 73.66 142.24 180)
+	(label "D-"
+		(at 33.02 144.78 0)
 		(effects
 			(font
 				(size 1.27 1.27)
 			)
-			(justify right bottom)
+			(justify left bottom)
 		)
 	)
-	(label "GPIO3"
-		(at 161.29 80.01 0)
+	(label "SYNC{slash}RESET"
+		(at 226.06 128.27 0)
 		(effects
 			(font
@@
 		)
 	)
-	(label "D-"
-		(at 33.02 144.78 0)
+	(label "GPIO4"
+		(at 227.33 60.96 0)
 		(effects
 			(font
@@
 	)
 	(label "5V_ISO"
-		(at 215.9 76.2 180)
+		(at 218.44 76.2 180)
 		(effects
 			(font
@@
 		)
 	)
+	(label "ESP_MOSI"
+		(at 226.06 109.22 0)
+		(effects
+			(font
+				(size 1.27 1.27)
+			)
+			(justify left bottom)
+		)
+	)
 	(label "5V_ISO"
 		(at 226.06 135.89 0)
@@
 		)
 	)
-	(label "GPIO4"
-		(at 161.29 83.82 0)
+	(label "ESP_MISO"
+		(at 158.75 95.25 0)
 		(effects
 			(font
@@
 		)
 	)
-	(label "ESP_MOSI"
-		(at 226.06 109.22 0)
+	(label "GPIO10"
+		(at 227.33 69.85 0)
+		(effects
+			(font
+				(size 1.27 1.27)
+			)
+			(justify left bottom)
+		)
+	)
+	(label "GPIO4"
+		(at 158.75 83.82 0)
 		(effects
 			(font
@@
 		)
 	)
-	(label "GPIO2"
-		(at 161.29 76.2 0)
+	(label "ESP_MISO"
+		(at 226.06 106.68 0)
 		(effects
 			(font
@@
 		)
 	)
+	(label "ESP_MOSI"
+		(at 158.75 76.2 0)
+		(effects
+			(font
+				(size 1.27 1.27)
+			)
+			(justify left bottom)
+		)
+	)
 	(label "ESP_TX"
-		(at 161.29 99.06 0)
+		(at 158.75 99.06 0)
 		(effects
 			(font
@@
 	(symbol
 		(lib_id "power:GNDA")
-		(at 208.28 80.01 90)
+		(at 210.82 80.01 90)
 		(unit 1)
 		(body_style 1)
@@
 		(fields_autoplaced yes)
 		(property "Reference" "#PWR037"
-			(at 214.63 80.01 0)
+			(at 217.17 80.01 0)
 			(hide yes)
 			(show_name no)
@@
 		)
 		(property "Value" "GNDA"
-			(at 212.09 80.0099 90)
+			(at 214.63 80.0099 90)
 			(show_name no)
 			(do_not_autoplace no)
@@
 		)
 		(property "Footprint" ""
-			(at 208.28 80.01 0)
+			(at 210.82 80.01 0)
 			(hide yes)
 			(show_name no)
@@
 		)
 		(property "Datasheet" ""
-			(at 208.28 80.01 0)
+			(at 210.82 80.01 0)
 			(hide yes)
 			(show_name no)
@@
 		)
 		(property "Description" "Power symbol creates a global label with name \"GNDA\" , analog ground"
-			(at 208.28 80.01 0)
+			(at 210.82 80.01 0)
 			(hide yes)
 			(show_name no)

Commit message: added Title & Rev
Other:
- company: (none) -> HAW-Hamburg
- title: (none) -> Reflectometer
Changed lines of the file:
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@@
 	(generator_version "10.0")
 	(paper "A4")
+	(title_block
+		(title "Reflectometer")
+		(rev "0.1")
+		(company "HAW-Hamburg")
+	)
 	(text "Strapping pins: GPIO2 - MOSI (should be high impedance input)\n		 		GPIO8 - SCLK (should be high impedance input)\n		 		GPIO9 - SYNC/RESET			(pulled high)\n				"
 		(exclude_from_sim no)
